Commit message: simulacion: etapa 2 (brazo y pinza con brazo_sim) y limoneros con las medidas de R1
Co-Authored-By: Claude Opus 5.5 <noreply@anthropic.com>

File: ros2_ws/src/simulacion/urdf/arturito.urdf.xacro (robot description, xacro)
@@ -1,4 +1,4 @@
 <?xml version="1.0"?>
-<!-- Arturito R2D2 en Gazebo Harmonic. Etapa 1: base diferencial con IMU y GPS (el brazo va en la etapa 2).
+<!-- Arturito R2D2 en Gazebo Harmonic: base diferencial con IMU y GPS + brazo RRR y pinza.
      Mismos marcos y tópicos que firmware/base: /cmd_vel, /odom (odom -> base_link), /imu/data_raw (imu_link),
      /gps/fix (gps_link). Radio y trocha de firmware/base/include/base_config.h; el chasis es una suposición (MEDIR). -->
@@ -119,3 +119,104 @@
     </plugin>
   </gazebo>
+  <!-- ===================== Brazo (etapa 2) =====================
+       Montado en la esquina delantera izquierda del chasis, junto a las ruedas; J1 = 0° mira al frente, paralelo al
+       costado (MEDIR la posición real). Medidas de la E4 (brazo_ik/cinematica.py). El cuatro barras se simula como
+       la cadena serie equivalente: j2 = q2 (hombro) y j3o = q3O (antebrazo respecto de la prolongación de l2);
+       brazo_sim convierte el actuador q3 <-> q3O. Articulaciones movidas por velocidad (JointPositionController con
+       use_velocity_commands): la gravedad no las afloja, como el sin fin de J2/J3. -->
+  <xacro:property name="brazo_x" value="${largo/2 - 0.05}"/>  <!-- MEDIR -->
+  <xacro:property name="brazo_y" value="${ancho/2 - 0.04}"/>  <!-- MEDIR -->
+  <xacro:property name="H1" value="0.150"/>
+  <xacro:property name="L2" value="0.35022"/>
+  <xacro:property name="L3" value="0.32951"/>
+  <xacro:property name="largo_pinza" value="0.11"/>  <!-- muñeca P3 -> punta de los dedos (MEDIR) -->
+  <xacro:property name="q2_ini" value="${pi/4}"/>          <!-- reposo de mision: q = (0°, 45°, 0°) -->
+  <xacro:property name="q3o_ini" value="-1.981223"/>       <!-- q3O = -113,516° para q2 = 45°, q3 = 0° (E4) -->
+  <xacro:macro name="barra" params="nombre largo_b ancho_b m color">
+    <link name="${nombre}">
+      <visual><origin xyz="${largo_b/2} 0 0"/><geometry><box size="${largo_b} ${ancho_b} ${ancho_b}"/></geometry>
+        <material name="${color}"/></visual>
+      <collision><origin xyz="${largo_b/2} 0 0"/><geometry><box size="${largo_b} ${ancho_b} ${ancho_b}"/></geometry></collision>
+      <inertial><origin xyz="${largo_b/2} 0 0"/><mass value="${m}"/>
+        <inertia ixx="${m*2*ancho_b*ancho_b/12}" iyy="${m*(largo_b*largo_b+ancho_b*ancho_b)/12}"
+                 izz="${m*(largo_b*largo_b+ancho_b*ancho_b)/12}" ixy="0" ixz="0" iyz="0"/></inertial>
+    </link>
+  </xacro:macro>
+  <link name="brazo_base"/>
+  <joint name="brazo_base_joint" type="fixed">
+    <parent link="base_link"/><child link="brazo_base"/><origin xyz="${brazo_x} ${brazo_y} ${alto}"/>
+  </joint>
+  <link name="torreta">
+    <visual><origin xyz="0 0 ${H1/2}"/><geometry><cylinder radius="0.04" length="${H1}"/></geometry>
+      <material name="naranja"><color rgba="0.9 0.45 0.1 1"/></material></visual>
+    <collision><origin xyz="0 0 ${H1/2}"/><geometry><cylinder radius="0.04" length="${H1}"/></geometry></collision>
+    <xacro:inercia_caja m="0.8" x="0.08" y="0.08" z="${H1}"/>
+  </link>
+  <joint name="j1" type="revolute">
+    <parent link="brazo_base"/><child link="torreta"/><axis xyz="0 0 1"/>
+    <limit lower="${radians(-75)}" upper="${radians(75)}" effort="50" velocity="1.0"/>
+  </joint>
+  <material name="verde"><color rgba="0.1 0.6 0.2 1"/></material>
+  <material name="azul"><color rgba="0.1 0.3 0.8 1"/></material>
+  <xacro:barra nombre="l2" largo_b="${L2}" ancho_b="0.03" m="0.5" color="verde"/>
+  <joint name="j2" type="revolute">
+    <!-- eje -y: q2 positivo levanta la barra (q2 desde la horizontal, como en la E4) -->
+    <parent link="torreta"/><child link="l2"/><origin xyz="0 0 ${H1}"/><axis xyz="0 -1 0"/>
+    <limit lower="${radians(-25)}" upper="${radians(135)}" effort="50" velocity="1.0"/>
+  </joint>
+  <xacro:barra nombre="l3" largo_b="${L3}" ancho_b="0.025" m="0.4" color="azul"/>
+  <joint name="j3o" type="revolute">
+    <parent link="l2"/><child link="l3"/><origin xyz="${L2} 0 0"/><axis xyz="0 -1 0"/>
+    <limit lower="${radians(-175)}" upper="${radians(10)}" effort="50" velocity="1.0"/>
+  </joint>
+  <!-- Pinza: giro J4 alrededor de l3 y dos dedos (servos RDS3218) -->
+  <link name="pinza">
+    <visual><origin xyz="0.02 0 0"/><geometry><box size="0.04 0.09 0.03"/></geometry><material name="gris"/></visual>
+    <collision><origin xyz="0.02 0 0"/><geometry><box size="0.04 0.09 0.03"/></geometry></collision>
+    <xacro:inercia_caja m="0.2" x="0.04" y="0.09" z="0.03"/>
+  </link>
+  <joint name="j4" type="revolute">
+    <parent link="l3"/><child link="pinza"/><origin xyz="${L3} 0 0"/><axis xyz="1 0 0"/>
+    <limit lower="${radians(-90)}" upper="${radians(90)}" effort="20" velocity="3.0"/>
+  </joint>
+  <xacro:macro name="dedo" params="lado signo">
+    <link name="dedo_${lado}">
+      <visual><origin xyz="${(largo_pinza - 0.04)/2} 0 0"/><geometry><box size="${largo_pinza - 0.04} 0.01 0.025"/></geometry>
+        <material name="negro"/></visual>
+      <!-- sin colisión: el agarre en la simulación se hará fijando el limón a la pinza al cerrar (etapa 4) -->
+      <xacro:inercia_caja m="0.05" x="${largo_pinza - 0.04}" y="0.01" z="0.025"/>
+    </link>
+    <!-- Sin gravedad: con la pinza girada, el control por velocidad de Gazebo no sostenía el peso de los dedos (uno
+         caía al tope); el servo real sí los sostiene -->
+    <gazebo reference="dedo_${lado}"><turnGravityOff>true</turnGravityOff></gazebo>
+    <joint name="dedo_${lado}_joint" type="prismatic">
+      <!-- 0 = cerrada; 0,035 m = abierta (cada dedo). PENDIENTE: con J4 girado los dedos quedan trabados en 0 o
+           0,035 (probado: gravedad, colisiones, límites, control por fuerza, masas; sin resolver). Con J4 = 0 andan -->
+      <parent link="pinza"/><child link="dedo_${lado}"/><origin xyz="0.04 ${signo*0.005} 0"/><axis xyz="0 ${signo} 0"/>
+      <limit lower="0" upper="0.035" effort="20" velocity="0.2"/>
+    </joint>
+  </xacro:macro>
+  <xacro:dedo lado="izq" signo="1"/>
+  <xacro:dedo lado="der" signo="-1"/>
+  <xacro:macro name="control_posicion" params="joint topico ini ganancia">
+    <plugin filename="gz-sim-joint-position-controller-system" name="gz::sim::systems::JointPositionController">
+      <joint_name>${joint}</joint_name>
+      <topic>${topico}</topic>
+      <use_velocity_commands>true</use_velocity_commands>
+      <p_gain>${ganancia}</p_gain>
+      <cmd_max>2.0</cmd_max>
+      <cmd_min>-2.0</cmd_min>
+      <initial_position>${ini}</initial_position>
+    </plugin>
+  </xacro:macro>
+  <gazebo>
+    <!-- brazo_sim publica en /sim/* consignas ya limitadas en velocidad (como el perfil del firmware) -->
+    <xacro:control_posicion joint="j1" topico="/sim/j1" ini="0" ganancia="10"/>
+    <xacro:control_posicion joint="j2" topico="/sim/j2" ini="${q2_ini}" ganancia="10"/>
+    <xacro:control_posicion joint="j3o" topico="/sim/j3o" ini="${q3o_ini}" ganancia="10"/>
+    <xacro:control_posicion joint="j4" topico="/sim/j4" ini="0" ganancia="10"/>
+    <!-- Un tópico por dedo: dos controladores en el mismo tópico no reciben los dos -->
+    <xacro:control_posicion joint="dedo_izq_joint" topico="/sim/dedo_izq" ini="0.035" ganancia="10"/>
+    <xacro:control_posicion joint="dedo_der_joint" topico="/sim/dedo_der" ini="0.035" ganancia="10"/>
+  </gazebo>
 </robot>

Commit message: simulacion: etapa 4 (agarre de limones y misión completa con visión simulada)
Co-Authored-By: Claude Opus 5.5 <noreply@anthropic.com>

File: ros2_ws/src/simulacion/urdf/arturito.urdf.xacro (robot description, xacro)
@@ -220,3 +220,34 @@
     <xacro:control_posicion joint="dedo_der_joint" topico="/sim/dedo_der" ini="0.035" ganancia="10"/>
   </gazebo>
+  <!-- ===================== Cámaras y agarre (etapa 4) =====================
+       stereo_camera_link = cámara izquierda (x adelante, z arriba), en un mástil del lado derecho mirando adelante a
+       la izquierda (55°) y un poco hacia abajo (MEDIR con el soporte rígido): mirando de costado (90°) veía limones
+       detrás del alcance de J1 (±75° desde el frente). "camera" es el marco óptico, con la misma rotación que publica
+       limon.launch.py de vision_estereo: /limon/posicion viene ahí. -->
+  <link name="stereo_camera_link"/>
+  <joint name="stereo_camera_joint" type="fixed">
+    <parent link="base_link"/><child link="stereo_camera_link"/>
+    <origin xyz="0.10 -0.10 ${alto + 0.30}" rpy="0 0.25 ${radians(55)}"/>
+  </joint>
+  <link name="camera"/>
+  <joint name="camera_optical_joint" type="fixed">
+    <parent link="stereo_camera_link"/><child link="camera"/><origin rpy="${-pi/2} 0 ${-pi/2}"/>
+  </joint>
+  <!-- Un enganche por limón cosechable (worlds/hilera.sdf): limones_sim publica en agarrar/soltar -->
+  <xacro:macro name="enganche" params="n">
+    <plugin filename="gz-sim-detachable-joint-system" name="gz::sim::systems::DetachableJoint">
+      <parent_link>pinza</parent_link>
+      <child_model>limon_${n}</child_model>
+      <child_link>link</child_link>
+      <attach_topic>/sim/limon_${n}/agarrar</attach_topic>
+      <detach_topic>/sim/limon_${n}/soltar</detach_topic>
+      <output_topic>/sim/limon_${n}/estado</output_topic>
+    </plugin>
+  </xacro:macro>
+  <gazebo>
+    <xacro:enganche n="1"/>
+    <xacro:enganche n="2"/>
+    <xacro:enganche n="3"/>
+    <xacro:enganche n="4"/>
+  </gazebo>
 </robot>

Commit message: simulacion: etapa 3 (cámaras de Gazebo + cadena real de visión), texturas y limones que aparecen con el brazo quieto
Co-Authored-By: Claude Opus 5.5 <noreply@anthropic.com>

File: ros2_ws/src/simulacion/urdf/arturito.urdf.xacro (robot description, xacro)
@@ -131,5 +131,8 @@
   <xacro:property name="L3" value="0.32951"/>
   <xacro:property name="largo_pinza" value="0.11"/>  <!-- muñeca P3 -> punta de los dedos (MEDIR) -->
-  <xacro:property name="q2_ini" value="${pi/4}"/>          <!-- reposo de mision: q = (0°, 45°, 0°) -->
+  <!-- Reposo: q = (-60°, 45°, 0°), el brazo estacionado hacia la derecha: con J1 = 0° la barra l2 tapaba los
+       limones en la cámara derecha y el estéreo no los localizaba -->
+  <xacro:property name="q1_ini" value="${radians(-60)}"/>
+  <xacro:property name="q2_ini" value="${pi/4}"/>
   <xacro:property name="q3o_ini" value="-1.981223"/>       <!-- q3O = -113,516° para q2 = 45°, q3 = 0° (E4) -->
   <xacro:macro name="barra" params="nombre largo_b ancho_b m color">
@@ -212,5 +215,5 @@
   <gazebo>
     <!-- brazo_sim publica en /sim/* consignas ya limitadas en velocidad (como el perfil del firmware) -->
-    <xacro:control_posicion joint="j1" topico="/sim/j1" ini="0" ganancia="10"/>
+    <xacro:control_posicion joint="j1" topico="/sim/j1" ini="${q1_ini}" ganancia="10"/>
     <xacro:control_posicion joint="j2" topico="/sim/j2" ini="${q2_ini}" ganancia="10"/>
     <xacro:control_posicion joint="j3o" topico="/sim/j3o" ini="${q3o_ini}" ganancia="10"/>
@@ -221,12 +224,17 @@
   </gazebo>
   <!-- ===================== Cámaras y agarre (etapa 4) =====================
-       stereo_camera_link = cámara izquierda (x adelante, z arriba), en un mástil del lado derecho mirando adelante a
-       la izquierda (55°) y un poco hacia abajo (MEDIR con el soporte rígido): mirando de costado (90°) veía limones
-       detrás del alcance de J1 (±75° desde el frente). "camera" es el marco óptico, con la misma rotación que publica
-       limon.launch.py de vision_estereo: /limon/posicion viene ahí. -->
+       stereo_camera_link = cámara izquierda (x adelante, z arriba), en un mástil detrás del brazo, del lado izquierdo,
+       a 0,55 m del piso, mirando 40° a la izquierda y 17° hacia abajo (MEDIR con el soporte rígido). El estéreo solo
+       localiza en la parte derecha de la imagen izquierda (u >= 271 px: con disparidad mínima 112 y rango 160, más a
+       la izquierda la búsqueda se sale de la imagen derecha): con el robot a x ~ 1 m, los 3 limones del árbol 1 caen
+       ahí, a 0,4-0,95 m y al alcance del brazo, y el brazo estacionado hacia la derecha queda fuera de la vista.
+       Probado antes: del lado derecho mirando de costado (90°) veía limones fuera del alcance de J1; a 55° la barra
+       l2 tapaba los limones en la cámara derecha; a 30° caían en la franja ciega del estéreo.
+       "camera" es el marco óptico, con la misma rotación que publica limon.launch.py de vision_estereo:
+       /limon/posicion viene ahí. -->
   <link name="stereo_camera_link"/>
   <joint name="stereo_camera_joint" type="fixed">
     <parent link="base_link"/><child link="stereo_camera_link"/>
-    <origin xyz="0.10 -0.10 ${alto + 0.30}" rpy="0 0.25 ${radians(55)}"/>
+    <origin xyz="-0.20 0.08 ${alto + 0.35}" rpy="0 0.30 ${radians(40)}"/>
   </joint>
   <link name="camera"/>
@@ -234,5 +242,30 @@
     <parent link="stereo_camera_link"/><child link="camera"/><origin rpy="${-pi/2} 0 ${-pi/2}"/>
   </joint>
-  <!-- Un enganche por limón cosechable (worlds/hilera.sdf): limones_sim publica en agarrar/soltar -->
+  <!-- Cámaras estéreo de Gazebo (etapa 3), solo con camaras:=true (renderizar es lo más pesado): como la calibración
+       v1, 640x480, f = 1076,5 px (33,1° de campo horizontal) y 99,26 mm de separación (Tx = -106,854). Imágenes
+       ideales, sin distorsión: salen directo como /left/image_rect y /right/image_rect (camara_info_sim les pone el
+       camera_info). La cámara derecha queda a la derecha de la izquierda (-y de stereo_camera_link). -->
+  <xacro:arg name="camaras" default="false"/>
+  <xacro:macro name="camara" params="nombre topico marco y">
+    <sensor name="${nombre}" type="camera">
+      <pose>0 ${y} 0 0 0 0</pose>
+      <always_on>true</always_on>
+      <update_rate>10</update_rate>
+      <topic>${topico}</topic>
+      <gz_frame_id>${marco}</gz_frame_id>
+      <camera>
+        <horizontal_fov>${2*atan(320/1076.537901)}</horizontal_fov>
+        <image><width>640</width><height>480</height><format>R8G8B8</format></image>
+        <clip><near>0.05</near><far>10</far></clip>
+      </camera>
+    </sensor>
+  </xacro:macro>
+  <xacro:if value="$(arg camaras)">
+    <gazebo reference="stereo_camera_link">
+      <xacro:camara nombre="cam_izq" topico="/left/image_rect" marco="camera" y="0"/>
+      <xacro:camara nombre="cam_der" topico="/right/image_rect" marco="camera_der" y="-0.099258"/>
+    </gazebo>
+  </xacro:if>
+  <!-- Un enganche por limón cosechable (12, config/limones_cosechables.xml): limones_sim publica en agarrar/soltar -->
   <xacro:macro name="enganche" params="n">
     <plugin filename="gz-sim-detachable-joint-system" name="gz::sim::systems::DetachableJoint">
@@ -243,4 +276,5 @@
       <detach_topic>/sim/limon_${n}/soltar</detach_topic>
       <output_topic>/sim/limon_${n}/estado</output_topic>
+      <suppress_child_warning>true</suppress_child_warning>  <!-- el limón aparece después (limones_sim) -->
     </plugin>
   </xacro:macro>
@@ -250,4 +284,12 @@
     <xacro:enganche n="3"/>
     <xacro:enganche n="4"/>
+    <xacro:enganche n="5"/>
+    <xacro:enganche n="6"/>
+    <xacro:enganche n="7"/>
+    <xacro:enganche n="8"/>
+    <xacro:enganche n="9"/>
+    <xacro:enganche n="10"/>
+    <xacro:enganche n="11"/>
+    <xacro:enganche n="12"/>
   </gazebo>
 </robot>

Commit message: Brazo tipo uArm: herramienta horizontal y TCP en brazo_ik, mision y simulación; limón llevado en el TCP
Co-Authored-By: Claude Opus 5.5 <noreply@anthropic.com>

File: ros2_ws/src/simulacion/urdf/arturito.urdf.xacro (robot description, xacro)
@@ -131,4 +131,5 @@
   <xacro:property name="L3" value="0.32951"/>
   <xacro:property name="largo_pinza" value="0.11"/>  <!-- muñeca P3 -> punta de los dedos (MEDIR) -->
+  <xacro:property name="largo_tcp" value="0.075"/>   <!-- muñeca P3 -> punto de agarre, entre los dedos (MEDIR); = largo_herramienta de brazo_ik -->
   <!-- Reposo: q = (-60°, 45°, 0°), el brazo estacionado hacia la derecha: con J1 = 0° la barra l2 tapaba los
        limones en la cámara derecha y el estéreo no los localizaba -->
@@ -173,5 +174,14 @@
     <limit lower="${radians(-175)}" upper="${radians(10)}" effort="50" velocity="1.0"/>
   </joint>
-  <!-- Pinza: giro J4 alrededor de l3 y dos dedos (servos RDS3218) -->
+  <!-- Brazo tipo uArm / Dobot Magician: un paralelogramo mantiene la herramienta horizontal, apuntando en la dirección
+       de J1 (E1). Se simula con j_nivel en la muñeca, al que brazo_sim le manda -(q2 + q3O) -->
+  <link name="muneca">
+    <inertial><mass value="0.05"/><inertia ixx="1e-5" iyy="1e-5" izz="1e-5" ixy="0" ixz="0" iyz="0"/></inertial>
+  </link>
+  <joint name="j_nivel" type="revolute">
+    <parent link="l3"/><child link="muneca"/><origin xyz="${L3} 0 0"/><axis xyz="0 -1 0"/>
+    <limit lower="${-pi}" upper="${pi}" effort="50" velocity="3.0"/>
+  </joint>
+  <!-- Pinza: giro J4 alrededor del eje de la herramienta (horizontal) y dos dedos (servos RDS3218) -->
   <link name="pinza">
     <visual><origin xyz="0.02 0 0"/><geometry><box size="0.04 0.09 0.03"/></geometry><material name="gris"/></visual>
@@ -180,5 +190,5 @@
   </link>
   <joint name="j4" type="revolute">
-    <parent link="l3"/><child link="pinza"/><origin xyz="${L3} 0 0"/><axis xyz="1 0 0"/>
+    <parent link="muneca"/><child link="pinza"/><axis xyz="1 0 0"/>
     <limit lower="${radians(-90)}" upper="${radians(90)}" effort="20" velocity="3.0"/>
   </joint>
@@ -194,12 +204,17 @@
     <gazebo reference="dedo_${lado}"><turnGravityOff>true</turnGravityOff></gazebo>
     <joint name="dedo_${lado}_joint" type="prismatic">
-      <!-- 0 = cerrada; 0,035 m = abierta (cada dedo). PENDIENTE: con J4 girado los dedos quedan trabados en 0 o
-           0,035 (probado: gravedad, colisiones, límites, control por fuerza, masas; sin resolver). Con J4 = 0 andan -->
+      <!-- 0 = cerrada; 0,045 m = abierta (cada dedo: entra un limón de 56 mm). La cara interna queda a la distancia
+           del prismático del eje de la herramienta -->
       <parent link="pinza"/><child link="dedo_${lado}"/><origin xyz="0.04 ${signo*0.005} 0"/><axis xyz="0 ${signo} 0"/>
-      <limit lower="0" upper="0.035" effort="20" velocity="0.2"/>
+      <limit lower="0" upper="0.045" effort="20" velocity="0.2"/>
     </joint>
   </xacro:macro>
   <xacro:dedo lado="izq" signo="1"/>
   <xacro:dedo lado="der" signo="-1"/>
+  <!-- Punto de agarre (TCP): ahí se engancha el limón y ahí apunta /brazo/objetivo -->
+  <link name="tcp"/>
+  <joint name="tcp_joint" type="fixed">
+    <parent link="pinza"/><child link="tcp"/><origin xyz="${largo_tcp} 0 0"/>
+  </joint>
   <xacro:macro name="control_posicion" params="joint topico ini ganancia">
     <plugin filename="gz-sim-joint-position-controller-system" name="gz::sim::systems::JointPositionController">
@@ -218,8 +233,9 @@
     <xacro:control_posicion joint="j2" topico="/sim/j2" ini="${q2_ini}" ganancia="10"/>
     <xacro:control_posicion joint="j3o" topico="/sim/j3o" ini="${q3o_ini}" ganancia="10"/>
+    <xacro:control_posicion joint="j_nivel" topico="/sim/j_nivel" ini="${-(q2_ini + q3o_ini)}" ganancia="10"/>
     <xacro:control_posicion joint="j4" topico="/sim/j4" ini="0" ganancia="10"/>
     <!-- Un tópico por dedo: dos controladores en el mismo tópico no reciben los dos -->
-    <xacro:control_posicion joint="dedo_izq_joint" topico="/sim/dedo_izq" ini="0.035" ganancia="10"/>
-    <xacro:control_posicion joint="dedo_der_joint" topico="/sim/dedo_der" ini="0.035" ganancia="10"/>
+    <xacro:control_posicion joint="dedo_izq_joint" topico="/sim/dedo_izq" ini="0.045" ganancia="10"/>
+    <xacro:control_posicion joint="dedo_der_joint" topico="/sim/dedo_der" ini="0.045" ganancia="10"/>
   </gazebo>
   <!-- ===================== Cámaras y agarre (etapa 4) =====================
@@ -267,29 +283,3 @@
     </gazebo>
   </xacro:if>
-  <!-- Un enganche por limón cosechable (12, config/limones_cosechables.xml): limones_sim publica en agarrar/soltar -->
-  <xacro:macro name="enganche" params="n">
-    <plugin filename="gz-sim-detachable-joint-system" name="gz::sim::systems::DetachableJoint">
-      <parent_link>pinza</parent_link>
-      <child_model>limon_${n}</child_model>
-      <child_link>link</child_link>
-      <attach_topic>/sim/limon_${n}/agarrar</attach_topic>
-      <detach_topic>/sim/limon_${n}/soltar</detach_topic>
-      <output_topic>/sim/limon_${n}/estado</output_topic>
-      <suppress_child_warning>true</suppress_child_warning>  <!-- el limón aparece después (limones_sim) -->
-    </plugin>
-  </xacro:macro>
-  <gazebo>
-    <xacro:enganche n="1"/>
-    <xacro:enganche n="2"/>
-    <xacro:enganche n="3"/>
-    <xacro:enganche n="4"/>
-    <xacro:enganche n="5"/>
-    <xacro:enganche n="6"/>
-    <xacro:enganche n="7"/>
-    <xacro:enganche n="8"/>
-    <xacro:enganche n="9"/>
-    <xacro:enganche n="10"/>
-    <xacro:enganche n="11"/>
-    <xacro:enganche n="12"/>
-  </gazebo>
 </robot>
