Commit message: simulacion: la base ya no se desliza con el brazo, pose real en limones_sim, perfil trapezoidal y obstáculos entre paradas
Co-Authored-By: Claude Opus 5.5 <noreply@anthropic.com>

File: ros2_ws/src/simulacion/urdf/arturito.urdf.xacro (robot description, xacro)
@@ -27,5 +27,5 @@
       <geometry><box size="${largo} ${ancho} ${alto}"/></geometry>
     </collision>
-    <xacro:inercia_caja m="8.0" x="${largo}" y="${ancho}" z="${alto}"/>
+    <xacro:inercia_caja m="20.0" x="${largo}" y="${ancho}" z="${alto}"/>
   </link>
   <xacro:macro name="rueda" params="lado signo">
@@ -127,4 +127,8 @@
   <xacro:property name="brazo_x" value="${largo/2 - 0.05}"/>  <!-- MEDIR -->
   <xacro:property name="brazo_y" value="${ancho/2 - 0.04}"/>  <!-- MEDIR -->
+  <!-- Masas del brazo al 5 %: las articulaciones se mueven por velocidad (fuerza ilimitada) y, con las masas reales,
+       cada movimiento hacía deslizar la base con las ruedas frenadas (~2-7 cm y 1,5-5° por movimiento). El brazo se
+       controla cinemáticamente (brazo_sim), así que su masa no se usa para nada más -->
+  <xacro:property name="k_masa" value="0.05"/>
   <xacro:property name="H1" value="0.150"/>
   <xacro:property name="L2" value="0.35022"/>
@@ -155,5 +159,5 @@
       <material name="naranja"><color rgba="0.9 0.45 0.1 1"/></material></visual>
     <collision><origin xyz="0 0 ${H1/2}"/><geometry><cylinder radius="0.04" length="${H1}"/></geometry></collision>
-    <xacro:inercia_caja m="0.8" x="0.08" y="0.08" z="${H1}"/>
+    <xacro:inercia_caja m="${0.8*k_masa}" x="0.08" y="0.08" z="${H1}"/>
   </link>
   <joint name="j1" type="revolute">
@@ -163,5 +167,5 @@
   <material name="verde"><color rgba="0.1 0.6 0.2 1"/></material>
   <material name="azul"><color rgba="0.1 0.3 0.8 1"/></material>
-  <xacro:barra nombre="l2" largo_b="${L2}" ancho_b="0.03" m="0.5" color="verde"/>
+  <xacro:barra nombre="l2" largo_b="${L2}" ancho_b="0.03" m="${0.5*k_masa}" color="verde"/>
   <joint name="j2" type="revolute">
     <!-- eje -y: q2 positivo levanta la barra (q2 desde la horizontal, como en la E4) -->
@@ -169,5 +173,5 @@
     <limit lower="${radians(-25)}" upper="${radians(135)}" effort="50" velocity="1.0"/>
   </joint>
-  <xacro:barra nombre="l3" largo_b="${L3}" ancho_b="0.025" m="0.4" color="azul"/>
+  <xacro:barra nombre="l3" largo_b="${L3}" ancho_b="0.025" m="${0.4*k_masa}" color="azul"/>
   <joint name="j3o" type="revolute">
     <parent link="l2"/><child link="l3"/><origin xyz="${L2} 0 0"/><axis xyz="0 -1 0"/>
@@ -177,5 +181,5 @@
        de J1 (E1). Se simula con j_nivel en la muñeca, al que brazo_sim le manda -(q2 + q3O) -->
   <link name="muneca">
-    <inertial><mass value="0.05"/><inertia ixx="1e-5" iyy="1e-5" izz="1e-5" ixy="0" ixz="0" iyz="0"/></inertial>
+    <inertial><mass value="${0.05*k_masa}"/><inertia ixx="${1e-5*k_masa}" iyy="${1e-5*k_masa}" izz="${1e-5*k_masa}" ixy="0" ixz="0" iyz="0"/></inertial>
   </link>
   <joint name="j_nivel" type="revolute">
@@ -187,5 +191,5 @@
     <visual><origin xyz="0.02 0 0"/><geometry><box size="0.04 0.09 0.03"/></geometry><material name="gris"/></visual>
     <collision><origin xyz="0.02 0 0"/><geometry><box size="0.04 0.09 0.03"/></geometry></collision>
-    <xacro:inercia_caja m="0.2" x="0.04" y="0.09" z="0.03"/>
+    <xacro:inercia_caja m="${0.2*k_masa}" x="0.04" y="0.09" z="0.03"/>
   </link>
   <joint name="j4" type="revolute">
@@ -198,5 +202,5 @@
         <material name="negro"/></visual>
       <!-- sin colisión: el agarre en la simulación se hará fijando el limón a la pinza al cerrar (etapa 4) -->
-      <xacro:inercia_caja m="0.05" x="${largo_pinza - 0.04}" y="0.01" z="0.025"/>
+      <xacro:inercia_caja m="${0.05*k_masa}" x="${largo_pinza - 0.04}" y="0.01" z="0.025"/>
     </link>
     <!-- Sin gravedad: con la pinza girada, el control por velocidad de Gazebo no sostenía el peso de los dedos (uno

Commit message: Base real (R2 E3) en firmware y simulación, batería de 36 V, 3 bumpers y docs reorganizados
- firmware/base: ruedas de 150 mm, trocha 0,40, 3 bumpers (frente y laterales), batería 10S (aviso a 32 V,
  divisor 120 k / 8,2 k)
- simulacion: caja en T con el brazo adelante a la izquierda y el mástil atrás; marcas y obstáculos
  recalculados: 12 de 12 limones cosechados
- docs: TPF R1/ y TPF R2/ sin carpetas repetidas, fotos/ (motor, pinza, rueda, batería), entregas nuevas en
  .md, INDICE, CONEXIONES (alimentación con 36 V, ubicación de la Pi y las cámaras)

Co-Authored-By: Claude Opus 5.5 <noreply@anthropic.com>

File: ros2_ws/src/simulacion/urdf/arturito.urdf.xacro (robot description, xacro)
@@ -2,13 +2,22 @@
 <!-- Arturito R2D2 en Gazebo Harmonic: base diferencial con IMU y GPS + brazo RRR y pinza.
      Mismos marcos y tópicos que firmware/base: /cmd_vel, /odom (odom -> base_link), /imu/data_raw (imu_link),
-     /gps/fix (gps_link). Radio y trocha de firmware/base/include/base_config.h; el chasis es una suposición (MEDIR). -->
+     /gps/fix (gps_link). Base de la R2 E3: caja de madera en T, 40 cm de largo; adelante la parte ancha (40 x 23 cm,
+     donde va el brazo), atrás la angosta (34 x 17 cm) con las ruedas de tracción en rebajes de 3 cm; paredes de 18 cm.
+     Ruedas inflables de 150 mm (docs/fotos/rueda). Lo marcado MEDIR es estimado. -->
 <robot name="arturito" xmlns:xacro="http://www.ros.org/wiki/xacro">
-  <xacro:property name="radio" value="0.05"/>     <!-- CFG_DIF.radioRueda (MEDIR) -->
-  <xacro:property name="trocha" value="0.30"/>    <!-- CFG_DIF.trocha (MEDIR) -->
-  <xacro:property name="ancho_rueda" value="0.04"/>
-  <xacro:property name="largo" value="0.50"/>     <!-- chasis (MEDIR) -->
-  <xacro:property name="ancho" value="0.24"/>     <!-- entre las ruedas -->
-  <xacro:property name="alto" value="0.15"/>
-  <xacro:property name="r_rueda_loca" value="0.025"/>
+  <xacro:property name="radio" value="0.075"/>      <!-- CFG_DIF.radioRueda: 150 mm, inflable (MEDIR con el inflado) -->
+  <xacro:property name="trocha" value="0.40"/>      <!-- CFG_DIF.trocha: entre centros de rueda (MEDIR) -->
+  <xacro:property name="ancho_rueda" value="0.045"/>
+  <xacro:property name="eje_atras" value="0.085"/>  <!-- eje: ranura centrada en el lateral de 17 cm (R2 E3, Lateral_Ejes) -->
+  <xacro:property name="largo_angosto" value="0.17"/>
+  <xacro:property name="ancho_angosto" value="0.34"/>
+  <xacro:property name="largo_ancho" value="0.23"/>
+  <xacro:property name="ancho_ancho" value="0.40"/>
+  <xacro:property name="alto_caja" value="0.20"/>   <!-- paredes de 18 cm + base y tapa de 1 cm -->
+  <xacro:property name="piso" value="0.03"/>        <!-- base de la caja sobre el piso: ranura del eje de 5 cm, ~2-3 cm (MEDIR) -->
+  <xacro:property name="abajo" value="${piso - radio}"/>        <!-- base de la caja respecto de base_link -->
+  <xacro:property name="alto" value="${abajo + alto_caja}"/>    <!-- tapa respecto de base_link (0,23 m del piso) -->
+  <xacro:property name="frente" value="${largo_angosto - eje_atras + largo_ancho}"/>  <!-- frente respecto del eje -->
+  <xacro:property name="r_rueda_loca" value="0.03"/>
   <xacro:macro name="inercia_caja" params="m x y z">
     <inertial><mass value="${m}"/>
@@ -16,16 +25,27 @@
     </inertial>
   </xacro:macro>
-  <!-- base_link en el centro del eje de las ruedas (a la altura del radio) -->
+  <!-- base_link en el centro del eje de las ruedas de tracción (atrás), a la altura del radio -->
   <link name="base_link">
     <visual>
-      <origin xyz="0 0 ${alto/2}"/>
-      <geometry><box size="${largo} ${ancho} ${alto}"/></geometry>
-      <material name="gris"><color rgba="0.5 0.5 0.55 1"/></material>
+      <origin xyz="${largo_angosto/2 - eje_atras} 0 ${abajo + alto_caja/2}"/>
+      <geometry><box size="${largo_angosto} ${ancho_angosto} ${alto_caja}"/></geometry>
+      <material name="gris"><color rgba="0.25 0.25 0.27 1"/></material>
+    </visual>
+    <visual>
+      <origin xyz="${frente - largo_ancho/2} 0 ${abajo + alto_caja/2}"/>
+      <geometry><box size="${largo_ancho} ${ancho_ancho} ${alto_caja}"/></geometry>
+      <material name="gris"/>
     </visual>
     <collision>
-      <origin xyz="0 0 ${alto/2}"/>
-      <geometry><box size="${largo} ${ancho} ${alto}"/></geometry>
+      <origin xyz="${largo_angosto/2 - eje_atras} 0 ${abajo + alto_caja/2}"/>
+      <geometry><box size="${largo_angosto} ${ancho_angosto} ${alto_caja}"/></geometry>
     </collision>
-    <xacro:inercia_caja m="20.0" x="${largo}" y="${ancho}" z="${alto}"/>
+    <collision>
+      <origin xyz="${frente - largo_ancho/2} 0 ${abajo + alto_caja/2}"/>
+      <geometry><box size="${largo_ancho} ${ancho_ancho} ${alto_caja}"/></geometry>
+    </collision>
+    <!-- 20 kg (MEDIR): madera, batería de 36 V, 2 motores de ~1 kg, drivers -->
+    <inertial><origin xyz="0.10 0 ${abajo + alto_caja/2}"/><mass value="20.0"/>
+      <inertia ixx="0.29" iyy="0.33" izz="0.53" ixy="0" ixz="0" iyz="0"/></inertial>
   </link>
   <xacro:macro name="rueda" params="lado signo">
@@ -40,6 +60,6 @@
         <geometry><cylinder radius="${radio}" length="${ancho_rueda}"/></geometry>
       </collision>
-      <inertial><mass value="0.6"/>
-        <inertia ixx="0.0004" iyy="0.00075" izz="0.0004" ixy="0" ixz="0" iyz="0"/>
+      <inertial><mass value="0.65"/>  <!-- 650 g por rueda -->
+        <inertia ixx="0.00102" iyy="0.00183" izz="0.00102" ixy="0" ixz="0" iyz="0"/>
       </inertial>
     </link>
@@ -53,27 +73,27 @@
   <xacro:rueda lado="izq" signo="1"/>
   <xacro:rueda lado="der" signo="-1"/>
-  <!-- Ruedas locas adelante y atrás, sin fricción -->
-  <xacro:macro name="rueda_loca" params="nombre x">
+  <!-- Dos ruedas locas bajo la parte ancha (adelante), sin fricción (MEDIR la posición) -->
+  <xacro:macro name="rueda_loca" params="nombre y">
     <link name="${nombre}">
       <visual><geometry><sphere radius="${r_rueda_loca}"/></geometry><material name="negro"/></visual>
       <collision><geometry><sphere radius="${r_rueda_loca}"/></geometry></collision>
-      <inertial><mass value="0.1"/><inertia ixx="2.5e-5" iyy="2.5e-5" izz="2.5e-5" ixy="0" ixz="0" iyz="0"/></inertial>
+      <inertial><mass value="0.1"/><inertia ixx="4e-5" iyy="4e-5" izz="4e-5" ixy="0" ixz="0" iyz="0"/></inertial>
     </link>
     <joint name="${nombre}_joint" type="fixed">
       <parent link="base_link"/>
       <child link="${nombre}"/>
-      <origin xyz="${x} 0 ${r_rueda_loca - radio}"/>
+      <origin xyz="${frente - 0.05} ${y} ${r_rueda_loca - radio}"/>
     </joint>
     <gazebo reference="${nombre}"><mu1>0.0</mu1><mu2>0.0</mu2></gazebo>
   </xacro:macro>
-  <xacro:rueda_loca nombre="rueda_loca_del" x="${largo/2 - 0.04}"/>
-  <xacro:rueda_loca nombre="rueda_loca_tras" x="${-largo/2 + 0.04}"/>
+  <xacro:rueda_loca nombre="rueda_loca_izq" y="0.13"/>
+  <xacro:rueda_loca nombre="rueda_loca_der" y="-0.13"/>
   <link name="imu_link"/>
   <joint name="imu_joint" type="fixed">
-    <parent link="base_link"/><child link="imu_link"/><origin xyz="0 0 0.05"/>
+    <parent link="base_link"/><child link="imu_link"/><origin xyz="0.10 0 ${abajo + 0.03}"/>
   </joint>
   <link name="gps_link"/>
   <joint name="gps_joint" type="fixed">
-    <parent link="base_link"/><child link="gps_link"/><origin xyz="-0.15 0 ${alto + 0.05}"/>
+    <parent link="base_link"/><child link="gps_link"/><origin xyz="0 -0.10 ${alto + 0.05}"/>
   </joint>
   <gazebo reference="imu_link">
@@ -120,11 +140,11 @@
   </gazebo>
   <!-- ===================== Brazo (etapa 2) =====================
-       Montado en la esquina delantera izquierda del chasis, junto a las ruedas; J1 = 0° mira al frente, paralelo al
-       costado (MEDIR la posición real). Medidas de la E4 (brazo_ik/cinematica.py). El cuatro barras se simula como
+       Montado adelante a la izquierda, sobre la parte ancha, a ~6 cm del frente y del costado (preliminar); J1 = 0°
+       mira al frente, paralelo al costado. Medidas de la E4 (brazo_ik/cinematica.py). El cuatro barras se simula como
        la cadena serie equivalente: j2 = q2 (hombro) y j3o = q3O (antebrazo respecto de la prolongación de l2);
        brazo_sim convierte el actuador q3 <-> q3O. Articulaciones movidas por velocidad (JointPositionController con
        use_velocity_commands): la gravedad no las afloja, como el sin fin de J2/J3. -->
-  <xacro:property name="brazo_x" value="${largo/2 - 0.05}"/>  <!-- MEDIR -->
-  <xacro:property name="brazo_y" value="${ancho/2 - 0.04}"/>  <!-- MEDIR -->
+  <xacro:property name="brazo_x" value="${frente - 0.06}"/>  <!-- adelante a la izquierda, a ~6 cm de cada borde (MEDIR) -->
+  <xacro:property name="brazo_y" value="${ancho_ancho/2 - 0.06}"/>
   <!-- Masas del brazo al 5 %: las articulaciones se mueven por velocidad (fuerza ilimitada) y, con las masas reales,
        cada movimiento hacía deslizar la base con las ruedas frenadas (~2-7 cm y 1,5-5° por movimiento). El brazo se
@@ -244,6 +264,6 @@
   </gazebo>
   <!-- ===================== Cámaras y agarre (etapa 4) =====================
-       stereo_camera_link = cámara izquierda (x adelante, z arriba), en un mástil detrás del brazo, del lado izquierdo,
-       a 0,55 m del piso, mirando 40° a la izquierda y 17° hacia abajo (MEDIR con el soporte rígido). El estéreo solo
+       stereo_camera_link = cámara izquierda (x adelante, z arriba), en un mástil atrás a la izquierda (detrás del
+       brazo), a 0,55 m del piso, mirando 40° a la izquierda y 17° hacia abajo (MEDIR con el soporte rígido). El estéreo solo
        localiza en la parte derecha de la imagen izquierda (u >= 271 px: con disparidad mínima 112 y rango 160, más a
        la izquierda la búsqueda se sale de la imagen derecha): con el robot a x ~ 1 m, los 3 limones del árbol 1 caen
@@ -256,5 +276,5 @@
   <joint name="stereo_camera_joint" type="fixed">
     <parent link="base_link"/><child link="stereo_camera_link"/>
-    <origin xyz="-0.20 0.08 ${alto + 0.35}" rpy="0 0.30 ${radians(40)}"/>
+    <origin xyz="-0.06 ${brazo_y} ${0.55 - radio}" rpy="0 0.30 ${radians(40)}"/>
   </joint>
   <link name="camera"/>

Commit message: simulacion: brazo atrás sobre el eje, mástil adelante a la derecha (dibujado) y brazo sin temblor
- Brazo sobre el eje de tracción a 6 cm del costado; mástil a (0,255; -0,17), cámara a 0,85 m mirando 94° y 28°
  abajo (buscado para ver y alcanzar los 3 limones de cada árbol); marcas en 1,19 / 2,70 / 4,17 / 5,69 m;
  reposo q = (-75°, 95°, -25°).
- Temblor: JointPositionController con use_velocity_commands va a la consigna en un paso (±1 rad/s y frenar);
  ahora JointController por velocidad (perfil + 5/s por el error) y /joint_states a 50 Hz (a 1 kHz ahogaba a
  los nodos de Python). 12 de 12 limones, 0 inversiones de velocidad.

Co-Authored-By: Claude Opus 5.5 <noreply@anthropic.com>

File: ros2_ws/src/simulacion/urdf/arturito.urdf.xacro (robot description, xacro)
@@ -137,14 +137,17 @@
     <plugin filename="gz-sim-joint-state-publisher-system" name="gz::sim::systems::JointStatePublisher">
       <topic>joint_states</topic>
+      <!-- sin esto sale en cada paso de física (1 kHz): ahogaba a los nodos de Python y la consigna del brazo llegaba
+           a saltos (temblor) -->
+      <update_rate>50</update_rate>
     </plugin>
   </gazebo>
   <!-- ===================== Brazo (etapa 2) =====================
-       Montado adelante a la izquierda, sobre la parte ancha, a ~6 cm del frente y del costado (preliminar); J1 = 0°
+       Montado atrás a la izquierda, sobre el eje de las ruedas de tracción, a ~6 cm del costado (preliminar); J1 = 0°
        mira al frente, paralelo al costado. Medidas de la E4 (brazo_ik/cinematica.py). El cuatro barras se simula como
        la cadena serie equivalente: j2 = q2 (hombro) y j3o = q3O (antebrazo respecto de la prolongación de l2);
        brazo_sim convierte el actuador q3 <-> q3O. Articulaciones movidas por velocidad (JointPositionController con
        use_velocity_commands): la gravedad no las afloja, como el sin fin de J2/J3. -->
-  <xacro:property name="brazo_x" value="${frente - 0.06}"/>  <!-- adelante a la izquierda, a ~6 cm de cada borde (MEDIR) -->
-  <xacro:property name="brazo_y" value="${ancho_ancho/2 - 0.06}"/>
+  <xacro:property name="brazo_x" value="0.0"/>  <!-- sobre el eje de tracción (MEDIR) -->
+  <xacro:property name="brazo_y" value="${ancho_angosto/2 - 0.06}"/>  <!-- a ~6 cm del costado izquierdo de la parte angosta -->
   <!-- Masas del brazo al 5 %: las articulaciones se mueven por velocidad (fuerza ilimitada) y, con las masas reales,
        cada movimiento hacía deslizar la base con las ruedas frenadas (~2-7 cm y 1,5-5° por movimiento). El brazo se
@@ -156,9 +159,4 @@
   <xacro:property name="largo_pinza" value="0.11"/>  <!-- muñeca P3 -> punta de los dedos (MEDIR) -->
   <xacro:property name="largo_tcp" value="0.075"/>   <!-- muñeca P3 -> punto de agarre, entre los dedos (MEDIR); = largo_herramienta de brazo_ik -->
-  <!-- Reposo: q = (-60°, 45°, 0°), el brazo estacionado hacia la derecha: con J1 = 0° la barra l2 tapaba los
-       limones en la cámara derecha y el estéreo no los localizaba -->
-  <xacro:property name="q1_ini" value="${radians(-60)}"/>
-  <xacro:property name="q2_ini" value="${pi/4}"/>
-  <xacro:property name="q3o_ini" value="-1.981223"/>       <!-- q3O = -113,516° para q2 = 45°, q3 = 0° (E4) -->
   <xacro:macro name="barra" params="nombre largo_b ancho_b m color">
     <link name="${nombre}">
@@ -252,10 +250,19 @@
     </plugin>
   </xacro:macro>
+  <!-- J1-J3 y el nivelador, por velocidad: brazo_sim manda la del perfil más una corrección del error. Con
+       JointPositionController (use_velocity_commands) Gazebo intentaba llegar a cada consigna en un paso de física
+       (±1 rad/s y frenar, 50 veces por segundo): el brazo temblaba -->
+  <xacro:macro name="control_velocidad" params="joint topico">
+    <plugin filename="gz-sim-joint-controller-system" name="gz::sim::systems::JointController">
+      <joint_name>${joint}</joint_name>
+      <topic>${topico}</topic>
+    </plugin>
+  </xacro:macro>
   <gazebo>
-    <!-- brazo_sim publica en /sim/* consignas ya limitadas en velocidad (como el perfil del firmware) -->
-    <xacro:control_posicion joint="j1" topico="/sim/j1" ini="${q1_ini}" ganancia="10"/>
-    <xacro:control_posicion joint="j2" topico="/sim/j2" ini="${q2_ini}" ganancia="10"/>
-    <xacro:control_posicion joint="j3o" topico="/sim/j3o" ini="${q3o_ini}" ganancia="10"/>
-    <xacro:control_posicion joint="j_nivel" topico="/sim/j_nivel" ini="${-(q2_ini + q3o_ini)}" ganancia="10"/>
+    <!-- Aparecen en 0 y brazo_sim las lleva al reposo -->
+    <xacro:control_velocidad joint="j1" topico="/sim/j1"/>
+    <xacro:control_velocidad joint="j2" topico="/sim/j2"/>
+    <xacro:control_velocidad joint="j3o" topico="/sim/j3o"/>
+    <xacro:control_velocidad joint="j_nivel" topico="/sim/j_nivel"/>
     <xacro:control_posicion joint="j4" topico="/sim/j4" ini="0" ganancia="10"/>
     <!-- Un tópico por dedo: dos controladores en el mismo tópico no reciben los dos -->
@@ -264,17 +271,37 @@
   </gazebo>
   <!-- ===================== Cámaras y agarre (etapa 4) =====================
-       stereo_camera_link = cámara izquierda (x adelante, z arriba), en un mástil atrás a la izquierda (detrás del
-       brazo), a 0,55 m del piso, mirando 40° a la izquierda y 17° hacia abajo (MEDIR con el soporte rígido). El estéreo solo
-       localiza en la parte derecha de la imagen izquierda (u >= 271 px: con disparidad mínima 112 y rango 160, más a
-       la izquierda la búsqueda se sale de la imagen derecha): con el robot a x ~ 1 m, los 3 limones del árbol 1 caen
-       ahí, a 0,4-0,95 m y al alcance del brazo, y el brazo estacionado hacia la derecha queda fuera de la vista.
-       Probado antes: del lado derecho mirando de costado (90°) veía limones fuera del alcance de J1; a 55° la barra
-       l2 tapaba los limones en la cámara derecha; a 30° caían en la franja ciega del estéreo.
+       stereo_camera_link = cámara izquierda (x adelante, z arriba), en un mástil adelante a la DERECHA, a 0,85 m del
+       piso, mirando 94° a la izquierda (de costado, hacia la fila, por encima del robot) y 28° hacia abajo (MEDIR con
+       el soporte rígido). El estéreo solo localiza en la parte derecha de la imagen izquierda (u >= 271 px: con
+       disparidad mínima 112 y rango 160, más a la izquierda la búsqueda se sale de la imagen derecha) y a 0,4-0,95 m.
+       Posición y ángulos buscados (brazo sobre el eje): para que desde cada marca de parada los 3 limones del árbol
+       caigan ahí y al alcance de J1 (±75°). Del lado izquierdo, pegada a la fila, quedaba demasiado cerca: los 3
+       limones ocupaban ~26° y la zona útil de la imagen tiene ~19°. Tolerancia de parada: ±2 cm.
        "camera" es el marco óptico, con la misma rotación que publica limon.launch.py de vision_estereo:
        /limon/posicion viene ahí. -->
-  <link name="stereo_camera_link"/>
+  <xacro:property name="mastil_x" value="${frente - 0.06}"/>          <!-- a ~6 cm del frente (MEDIR) -->
+  <xacro:property name="mastil_y" value="${-(ancho_ancho/2 - 0.03)}"/> <!-- a ~3 cm del costado derecho (MEDIR) -->
+  <xacro:property name="mastil_alto" value="0.85"/>                    <!-- cámara izquierda sobre el piso (MEDIR) -->
+  <!-- Mástil y cámaras dibujados (solo visual): para ver si el brazo las tapa o las toca al moverse -->
+  <link name="mastil">
+    <visual><origin xyz="0 0 ${(mastil_alto - radio - alto)/2}"/>
+      <geometry><cylinder radius="0.012" length="${mastil_alto - radio - alto}"/></geometry>
+      <material name="gris"/></visual>
+  </link>
+  <joint name="mastil_joint" type="fixed">
+    <parent link="base_link"/><child link="mastil"/><origin xyz="${mastil_x} ${mastil_y} ${alto}"/>
+  </joint>
+  <link name="stereo_camera_link">
+    <!-- barra de las cámaras (99 mm entre ejes) y los dos "ojos", mirando por +x -->
+    <visual><origin xyz="-0.015 -0.0496 0"/><geometry><box size="0.02 0.14 0.02"/></geometry>
+      <material name="negro"/></visual>
+    <visual><origin xyz="0.005 0 0" rpy="0 ${pi/2} 0"/><geometry><cylinder radius="0.01" length="0.02"/></geometry>
+      <material name="azul"/></visual>
+    <visual><origin xyz="0.005 -0.099258 0" rpy="0 ${pi/2} 0"/><geometry><cylinder radius="0.01" length="0.02"/></geometry>
+      <material name="azul"/></visual>
+  </link>
   <joint name="stereo_camera_joint" type="fixed">
     <parent link="base_link"/><child link="stereo_camera_link"/>
-    <origin xyz="-0.06 ${brazo_y} ${0.55 - radio}" rpy="0 0.30 ${radians(40)}"/>
+    <origin xyz="${mastil_x} ${mastil_y} ${mastil_alto - radio}" rpy="0 ${radians(28)} ${radians(94)}"/>
   </joint>
   <link name="camera"/>
