Commit message: J1: rango 45°/225° en el marco de brazo_ik (cero al costado izquierdo = 90°)
Decisión del usuario: en el banco de pruebas el cero de J1 es el brazo al costado izquierdo
y el rango -45/+135 desde ahí. En el marco de la cinemática (q1 = 0 al frente, antihorario)
eso es 45°..225°: pasa por atrás y no cruza el mástil (adelante-derecha).

- brazo_config.h: qMin/qMax 45/225, POSE_CERO J1 = 90, HOME_Q J1 = 45 (MEDIR)
- cinematica.py: Q1_LIM y q1_en_rango() (atan2 da -180..180 y el rango pasa por 180°)
- urdf: límites de j1
- fsm.py: reposo por defecto = el de la simulación (el anterior, al frente, quedó afuera)
- Pruebas con puntos al frente giradas al costado izquierdo; una nueva para q1 = 200°
- Pruebas: firmware 17, brazo_ik 7, mision 27, simulacion 13 OK. Sin probar en Gazebo

File: ros2_ws/src/simulacion/urdf/arturito.urdf.xacro (robot description, xacro)
@@ -239,5 +239,5 @@
   <joint name="j1" type="revolute">
     <parent link="brazo_base"/><child link="torreta"/><axis xyz="0 0 1"/>
-    <limit lower="${radians(-75)}" upper="${radians(75)}" effort="50" velocity="1.0"/>
+    <limit lower="${radians(45)}" upper="${radians(225)}" effort="50" velocity="1.0"/>
   </joint>
   <material name="verde"><color rgba="0.1 0.6 0.2 1"/></material>
